File: KiCAD_Camsat_PCB/KiCAD_Camsat_PCB.kicad_pcb (KiCad board)
At the start: 2 copper layers, 70 x 136.3 mm, 64 parts, among them J1 Barrel_Jack, J3 105017-0001, K1 HYC77-TF09-200, Q2 SS8050-G_C164885, Q9 SS8050-G_C164885, U1 ISM330DHCX, U10 BME280, U5 DHT11, U6 LM2596S-5, U7 AMS1117-3.3_C347222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

Commit message: Generate Gerber Files
Parts:
- moved J1 2.00 mm to (79.0, 51.5)
Routing:
- net /9V: track 11.2 -> 10.3 mm
- net GND: vias 129 -> 143

Commit message: PCB Footprint + layout changes
Parts:
- C14: value 470uF -> 220uF; footprint Capacitor_SMD:C_0603_1608Metric -> Capacitor_SMD:CP_Elec_6.3x5.4
- C15: value 470uF -> 330uF; footprint Capacitor_SMD:C_0603_1608Metric -> Capacitor_SMD:CP_Elec_6.3x5.4
- LED2: renamed from Debug LED
- moved C14 9.65 mm to (61.5, 53.5)
- moved L1 3.15 mm to (57.5, 62.8)
- moved J1 2.46 mm to (76.8, 50.5)
- moved C15 1.43 mm to (59.5, 71.5), turned to 0 degrees
- moved D8 0.80 mm to (56.0, 77.8)
- moved D5 0.70 mm to (66.2, 63.1)
- renumbered Reset to SW1, Boot to SW2
Connections:
- C14 pad 1: GND -> /9VIN
- C14 pad 2: /9VIN -> GND
- C15 pad 1: GND -> /5V_Board
- C15 pad 2: /5V_Board -> GND
Routing:
- net /9VIN: track 0.00 -> 5.48 mm
- net /9V: track 10.3 -> 8.33 mm
Other:
- board text added: "Boot"
- board text added: "Debug"
- board text added: "Reset"
