File: KiCAD_Camsat_PCB/KiCAD_Camsat_PCB.kicad_sch (KiCad schematic)
At the start: 62 parts, among them J1 Barrel_Jack, J3 105017-0001, K1 HYC77-TF09-200, Q2 SS8050-G_C164885, Q9 SS8050-G_C164885, SW1 PTS645SH50SMTR92LFS, SW2 PTS645SH50SMTR92LFS, U1 ISM330DHCX, U10 BME280, U5 DHT11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

Commit message: PCB Footprint + layout changes
Parts:
- C14: value 470uF -> 220uF; footprint Capacitor_SMD:C_0603_1608Metric -> Capacitor_SMD:CP_Elec_6.3x5.4
- C15: value 470uF -> 330uF; footprint Capacitor_SMD:C_0603_1608Metric -> Capacitor_SMD:CP_Elec_6.3x5.4
Connections:
- net 5V_Board: now also C15.1 (2); no longer C15.2
- net 9VIN: now also C14.1 (2); no longer C14.2
- net GND: now also C14.2 (1), C15.2 (1); no longer C14.1, C15.1
